File: omega_hotswap/omega.kicad_pcb (KiCad board)
At the start: 2 copper layers, 200.8 x 58.9 mm, 61 parts, among them SW1 SW_Push, U1 ProMicro

Commit message: work
Parts:
- added H1: MountingHole, MountingHole:MountingHole_2.2mm_M2_Pad, F.Cu at (232.3, 60.5)
- added H2: MountingHole, MountingHole:MountingHole_2.2mm_M2_Pad, F.Cu at (79.9, 61.9)
- added H3: MountingHole, MountingHole:MountingHole_2.2mm_M2_Pad, F.Cu at (232.2, 79.5)
- added H4: MountingHole, MountingHole:MountingHole_2.2mm_M2_Pad, F.Cu at (79.8, 79.5)
- D1, D10, D11, D12, D13, D14, D15, D16, D17, D18, D19, D2, D20, D21, D22, D23, D24, D25, D26, D27, D28, D29, D3, D4, D5, D6, D7, D8, D9: footprint Diode_THT:D_DO-35_SOD27_P3.81mm_Vertical_AnodeUp -> Keebio-Parts:Diode-Hybrid-Back; moved to F.Cu
- moved D26 4.63 mm to (197.5, 91.4), turned to 270 degrees
- moved D7 4.62 mm to (188.0, 53.3), turned to 270 degrees
- moved D9 4.62 mm to (226.1, 53.3), turned to 270 degrees
- moved D6 4.62 mm to (168.9, 53.3), turned to 270 degrees
- moved D14 4.59 mm to (135.5, 72.4), turned to 270 degrees
- moved D18 4.59 mm to (211.7, 72.4), turned to 270 degrees
- moved D22 4.59 mm to (102.3, 91.5), turned to 270 degrees
- moved D3 4.57 mm to (111.8, 53.4), turned to 270 degrees
- moved D4 4.57 mm to (130.8, 53.4), turned to 270 degrees
- moved D8 4.57 mm to (207.0, 53.4), turned to 270 degrees
- moved D24 4.57 mm to (140.4, 91.4), turned to 270 degrees
- moved D15 4.56 mm to (154.5, 72.4), turned to 270 degrees
- moved D27 4.56 mm to (216.5, 91.5), turned to 270 degrees
- moved D28 4.56 mm to (235.6, 91.5), turned to 270 degrees
- moved D23 4.55 mm to (121.4, 91.5), turned to 270 degrees
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Routing:
- net Net-(D19-Pad2): track 9.29 -> 4.19 mm
- net Net-(D11-Pad2): track 9.29 -> 4.20 mm
- net Net-(D10-Pad2): track 8.98 -> 4.37 mm
- net Net-(D2-Pad2): track 8.57 -> 4.22 mm
- net Net-(D29-Pad2): track 9.50 -> 5.37 mm
- net Net-(D26-Pad2): track 9.50 -> 5.45 mm
- net Net-(D24-Pad2): track 9.50 -> 5.45 mm
- net Net-(D27-Pad2): track 9.50 -> 5.48 mm
- net Net-(D28-Pad2): track 9.50 -> 5.48 mm
- net Net-(D22-Pad2): track 9.50 -> 5.50 mm
- net Net-(D23-Pad2): track 9.50 -> 5.52 mm
- net Net-(D21-Pad2): track 9.39 -> 5.48 mm
- net Net-(D13-Pad2): track 9.29 -> 5.43 mm
- net Net-(D12-Pad2): track 9.29 -> 5.43 mm
- net ROW0: track 175.0 -> 178.8 mm
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Other:
- board text added: "omega_v2"
- board text removed: "omega_v0"
